Commit message: 1

File: pybullet/urdf/simplearm.urdf (robot description, URDF)
Before this commit: robot arm, 3 links, 2 joints
Links:
- link big_arm: geometry collision cylinder length=0.6 radius=0.05; visual cylinder length=0.6 radius=0.05
- link small_arm: geometry collision cylinder length=0.4 radius=0.04; visual cylinder length=0.4 radius=0.04
Joints:
- joint elbow: origin xyz=0.0 0.0 0.25 -> xyz=0.0 0.0 0.30
- joint wrist: origin xyz=0.0 0.0 0.15 -> xyz=0.0 0.0 0.25
